Commit message: openDog geometry

File: urdf/lidar_body.urdf (robot description, URDF)
Before this commit: robot lidar_body, 4 links, 3 joints
Links:
- link base_link: geometry collision box size=0.9 0.4 0.74; visual box size=0.9 0.23 0.74
Joints:
- joint base_link_joint: origin xyz=0.0 0 1.25 rpy=0 0 0 -> xyz=0.0 0.0 0.37 rpy=0 0 0
- joint camera_joint: parent base_link -> base_footprint
- joint laser_joint: axis 0 1 0 -> 0 0 0; parent base_link -> base_footprint

Commit message: added bumper to robot model

File: urdf/lidar_body.urdf (robot description, URDF)
Before this commit: robot lidar_body, 4 links, 3 joints
Links:
- link base_link: geometry collision box size=0.9 0.4 0.5; visual box size=0.9 0.23 0.74

Commit message: Update lidar_body.urdf

File: urdf/lidar_body.urdf (robot description, URDF)
Before this commit: robot lidar_body, 4 links, 3 joints
Links:
- link base_link: geometry collision box size=0.9 0.4 0.74; visual box size=0.9 0.23 0.74
